File: meteo/esp8266_test_board.sch (KiCad schematic (older format))
At the start: 31 parts, among them J1 USB-MINI-B-SMD, K1 CONN_3, P1 Solar, P10 DRILL, P12 DRILL, P2 CONN_6, P3 CONN_7, P8 NIMH 1.2V, P9 DRILL, SW1 RST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

Commit message: -
Other:
- note added: "Voltage selector\nNC -> 2.5V \ngnd ->3V\nVCC ->3.3V"
- moved on the sheet: C1, C2, C3, C4, C5, C6, C7, D1, D2, D3, J1, K1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
